File: Pride Badge.sch (KiCad schematic (older format))
At the start: 0 parts

Commit message: Prototype PCB design finished?
Changed lines of the file:
@@
 F0 "SheetPower" 50
 F1 "power.sch" 50
-F2 "USB_D+" I L 3550 2600 50
-F3 "USB_D-" I L 3550 2700 50
-F4 "VUSB" I L 3550 2500 50
-F5 "VBATT" I R 4400 2500 50
-F6 "GND" I R 4400 2800 50
-F7 "5V" I R 4400 2600 50
-F8 "3V3" I R 4400 2700 50
-$EndSheet
-$Sheet
-S 4950 2400 950  500
-U 5B33D5D4
-F0 "Sheet_MCU-LED-Driver" 50
-F1 "MCU_LED-Driver.sch" 50
-F2 "5V" I R 5900 2500 50
-F3 "GND" I R 5900 2700 50
-F4 "USB_D+" I L 4950 2500 50
-F5 "USB_D-" I L 4950 2600 50
-F6 "3V3" I R 5900 2600 50
+F2 "VUSB" O L 3550 2500 50
+F3 "VBATT" O R 4400 2500 50
+F4 "GND" O R 4400 2800 50
+F5 "5V" O R 4400 2600 50
+F6 "3V3" O R 4400 2700 50
 $EndSheet
 $Sheet
@@
 F4 "GND" I L 4200 3450 50
 $EndSheet
+$Sheet
+S 4950 2400 950  500
+U 5B33D5D4
+F0 "Sheet_MCU-LED-Driver" 50
+F1 "MCU_LED-Driver.sch" 50
+F2 "5V" U R 5900 2500 50
+F3 "GND" U R 5900 2700 50
+F4 "3V3" U R 5900 2600 50
+$EndSheet
 $EndSCHEMATC
