File: Pride Badge.kicad_pcb (KiCad board)
At the start: 2 copper layers, 100 x 130 mm, 93 parts, among them J1 USB_B_Micro, J2 Conn_Batt_JST-PH, J3 SWD, J4 SWD20, SW1 PWR_SW, SW2 Mode_BTN, SW3 Bright_BTN, SW4 Reset_BTN, SW5 Boot_SW, SW6 SW_SeeBattGauge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

Commit message: Fixed up PCB design after fixing some IC footprints
Parts:
- C14: value 1u -> 1uF
- C15: value 100n -> 100nF
- C4: value 22uF -> 22u
- D3: value 2V5 Z -> 2V5 Zener
- J3: value SWD -> SWD_Conn
- J4: value SWD20 -> Conn_SWD20
- R7: value 100R -> 100
- SW1: footprint digikey-footprints:Switch_Slide_JS202011SCQN -> my-footprints:Switch_Slide_JS202011SCQN
- U7: footprint digikey-footprints:SOIC-24_W7.50mm -> digikey-footprints:TSSOP-20_W4.4mm
- U8: footprint SMD_Packages:SOIC-24 -> digikey-footprints:SOIC-24_W7.50mm
- U9: footprint digikey-footprints:SOIC-24_W7.50mm -> digikey-footprints:SOIC-14_W3.9mm
- moved U7 5.61 mm to (50.5, 88.8)
- moved U8 0.90 mm to (78.3, 82.3)
- moved U9 0.45 mm to (90.3, 50.1)
Routing:
- net Net-(R16-Pad2): track 17.5 -> 37.9 mm, vias 0 -> 2
- net Net-(R20-Pad2): track 7.03 -> 21.6 mm, vias 0 -> 2
- net Net-(SW5-Pad2): track 7.85 -> 18.6 mm
- net +5V: track 318.8 -> 308.7 mm, vias 0 -> 2
- net /Sheet_MCU-LED-Driver/SDA0: track 38.0 -> 48.1 mm
- net +3V3: track 241.7 -> 232.1 mm
- net /Sheet_MCU-LED-Driver/RESET: track 104.5 -> 114.1 mm
- net Net-(DF1-Pad1): track 32.3 -> 23.9 mm
- net Net-(D7-Pad1): track 4.43 -> 12.7 mm
- net /Sheet_MCU-LED-Driver/SCL0: track 36.9 -> 44.6 mm
- net GND: track 110.5 -> 104.9 mm
- net Net-(D3-Pad1): track 32.1 -> 37.4 mm
- net /Sheet_MCU-LED-Driver/SWDIO: track 30.7 -> 34.8 mm
- net Net-(DE3-Pad1): track 59.8 -> 55.8 mm
- net Net-(D6-Pad1): track 10.5 -> 6.57 mm
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Other:
- board text added: "OFF"
- board text added: "ON"
