File: Pride Badge.kicad_pcb (KiCad board)
At the start: 2 copper layers, 93 parts, among them J1 USB_B_Micro, J2 Conn_Batt_JST-PH, J3 SWD_Conn, J4 Conn_SWD20, SW1 PWR_SW, SW2 Mode_BTN, SW3 Bright_BTN, SW4 Reset_BTN, SW5 Boot_SW, SW6 SW_SeeBattGauge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

Commit message: Prototype PCB design finished?
Parts:
- C14: value 1uF -> 1u
- C15: value 100nF -> 100n
- C4: value 22u -> 22uF
- D3: value 2V5 Zener -> 2V5 Z
- J3: value SWD_Conn -> SWD
- J4: value Conn_SWD20 -> SWD20
- R7: value 100 -> 100R
- moved J2 21.5 mm to (105.3, 117.2), turned to 270 degrees
- moved R2 19.4 mm to (66.1, 114.1)
- moved C3 19.4 mm to (62.6, 120.6)
- moved C6 19.4 mm to (57.4, 137.5)
- moved L1 19.4 mm to (58.4, 117.3)
- moved U1 19.4 mm to (48.6, 120.6)
- moved U4 19.4 mm to (57.1, 131.4)
- moved C4 19.4 mm to (83.0, 144.1)
- moved C7 19.4 mm to (51.5, 131.5)
- moved D1 19.4 mm to (96.7, 138.2)
- moved F1 19.4 mm to (81.0, 137.5)
- moved L2 19.4 mm to (87.5, 135.2)
- moved R3 19.4 mm to (67.5, 126.8)
- moved R4 19.4 mm to (93.0, 142.2)
- moved R5 19.4 mm to (68.9, 114.0)
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Connections:
- D2 pad 1: /SheetPower/VUSB -> Net-(C2-Pad1)
- D2 pad 2: /SheetPower/VUSB -> Net-(C2-Pad1)
- U1 pad 4: (no net) -> USBDM
- U1 pad 6: (no net) -> USBDP
- U7 pad 17: (no net) -> USBDP
- U7 pad 18: (no net) -> USBDM
Routing:
- net +5V: track 0.00 -> 318.8 mm
- net +3V3: track 0.00 -> 241.7 mm, vias 0 -> 2
- net +BATT: track 0.00 -> 166.4 mm, vias 0 -> 4
- net GND: track 0.00 -> 110.5 mm, vias 0 -> 11
- net /Sheet_MCU-LED-Driver/RESET: track 0.00 -> 104.5 mm
- net Net-(DC2-Pad1): track 0.00 -> 96.6 mm
- net Net-(DD1-Pad1): track 0.00 -> 93.4 mm
- net Net-(DC3-Pad1): track 0.00 -> 85.6 mm
- net Net-(DD2-Pad1): track 0.00 -> 82.6 mm
- net Net-(DE1-Pad1): track 0.00 -> 79.7 mm
- net Net-(DD3-Pad1): track 0.00 -> 71.0 mm
- net Net-(DE2-Pad1): track 0.00 -> 69.6 mm
- net Net-(DE3-Pad1): track 0.00 -> 59.8 mm
- net /SheetBatteryGauge/LED_VCC: track 0.00 -> 54.9 mm
- net Net-(DB3-Pad1): track 0.00 -> 53.1 mm
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- added copper zone on F.Cu, net +5V
Other:
- board outline added: 100 x 159.9 mm
- net class Default: clearance 0.2 -> 0.3; via_dia 0.8 -> 2; via_drill 0.4 -> 1
- rule trace_clearance: 0.2 -> 0.3
- rule trace_min: 0.2 -> 0.25
- rule via_min_drill: 0.3 -> 0.1
- rule via_min_size: 0.4 -> 0.2
- board text added: "- Batt +"
- board text added: "1"
- board text added: "3V3"
- board text added: "5V"
- board text added: "Boot"
- board text added: "Bootloader"
- board text added: "Bright"
- board text added: "D+"
- board text added: "D-"
- board text added: "GND"
- board text added: "Mode"
- board text added: "Normal"
- board text added: "Reset"
- board text added: "SC"
- board text added: "SD"
- board text added: "Show Batt Level"
- board text added: "USB"
- board text added: "Vbatt"

Commit message: Prototype PCB gerbers plotted & PCB layout tweaked
Other:
- board size 100 x 159.9 mm -> 100 x 130 mm
Changed lines of the file:
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@@
   (general
     (thickness 1.6)
-    (drawings 30)
+    (drawings 26)
     (tracks 853)
     (zones 0)
@@
     (visible_elements 7FFFFF7F)
     (pcbplotparams
-      (layerselection 0x010fc_ffffffff)
+      (layerselection 0x01000_7fffffff)
       (usegerberextensions false)
       (usegerberattributes false)
@@
       (outputformat 1)
       (mirror false)
-      (drillshape 1)
+      (drillshape 0)
       (scaleselection 1)
-      (outputdirectory ""))
+      (outputdirectory "gerbers"))
   )
   (net 0 "")
@@
     (effects (font (size 1 1) (thickness 0.15)) (justify right))
   )
-  (gr_line (start 27.7 176.45) (end 27.7 16.5) (layer Edge.Cuts) (width 0.2))
-  (gr_line (start 127.7 176.45) (end 27.7 176.45) (layer Edge.Cuts) (width 0.2))
-  (gr_line (start 127.7 16.5) (end 127.7 176.45) (layer Edge.Cuts) (width 0.2))
-  (gr_line (start 27.7 16.5) (end 127.7 16.5) (layer Edge.Cuts) (width 0.2))
+  (gr_line (start 27.7 150.4) (end 27.7 20.399962) (layer Edge.Cuts) (width 0.2))
+  (gr_line (start 127.7 150.4) (end 27.7 150.4) (layer Edge.Cuts) (width 0.2))
+  (gr_line (start 127.7 20.4) (end 127.7 150.4) (layer Edge.Cuts) (width 0.2))
+  (gr_line (start 27.7 20.4) (end 127.700012 20.4) (layer Edge.Cuts) (width 0.2))
   (gr_text SD (at 47.65 71.75) (layer F.Cu)
     (effects (font (size 1 1) (thickness 0.15)))
@@
     (effects (font (size 1.5 1.5) (thickness 0.15)))
   )
-  (gr_line (start 127.7 176.45) (end 127.7 16.5) (layer F.SilkS) (width 0.2))
-  (gr_line (start 27.7 176.45) (end 127.7 176.45) (layer F.SilkS) (width 0.2))
-  (gr_line (start 27.7 16.5) (end 27.7 176.45) (layer F.SilkS) (width 0.2))
-  (gr_line (start 127.7 16.5) (end 27.7 16.5) (layer F.SilkS) (width 0.2))
   (segment (start 69.6 74.35) (end 69.6 71.7) (width 0.25) (layer F.Cu) (net 1))
   (segment (start 69.6 71.7) (end 75.6 65.7) (width 0.25) (layer F.Cu) (net 1))

Commit message: Fixed up PCB design after fixing some IC footprints
Parts:
- C14: value 1u -> 1uF
- C15: value 100n -> 100nF
- C4: value 22uF -> 22u
- D3: value 2V5 Z -> 2V5 Zener
- J3: value SWD -> SWD_Conn
- J4: value SWD20 -> Conn_SWD20
- R7: value 100R -> 100
- SW1: footprint digikey-footprints:Switch_Slide_JS202011SCQN -> my-footprints:Switch_Slide_JS202011SCQN
- U7: footprint digikey-footprints:SOIC-24_W7.50mm -> digikey-footprints:TSSOP-20_W4.4mm
- U8: footprint SMD_Packages:SOIC-24 -> digikey-footprints:SOIC-24_W7.50mm
- U9: footprint digikey-footprints:SOIC-24_W7.50mm -> digikey-footprints:SOIC-14_W3.9mm
- moved U7 5.61 mm to (50.5, 88.8)
- moved U8 0.90 mm to (78.3, 82.3)
- moved U9 0.45 mm to (90.3, 50.1)
Routing:
- net Net-(R16-Pad2): track 17.5 -> 37.9 mm, vias 0 -> 2
- net Net-(R20-Pad2): track 7.03 -> 21.6 mm, vias 0 -> 2
- net Net-(SW5-Pad2): track 7.85 -> 18.6 mm
- net +5V: track 318.8 -> 308.7 mm, vias 0 -> 2
- net /Sheet_MCU-LED-Driver/SDA0: track 38.0 -> 48.1 mm
- net +3V3: track 241.7 -> 232.1 mm
- net /Sheet_MCU-LED-Driver/RESET: track 104.5 -> 114.1 mm
- net Net-(DF1-Pad1): track 32.3 -> 23.9 mm
- net Net-(D7-Pad1): track 4.43 -> 12.7 mm
- net /Sheet_MCU-LED-Driver/SCL0: track 36.9 -> 44.6 mm
- net GND: track 110.5 -> 104.9 mm
- net Net-(D3-Pad1): track 32.1 -> 37.4 mm
- net /Sheet_MCU-LED-Driver/SWDIO: track 30.7 -> 34.8 mm
- net Net-(DE3-Pad1): track 59.8 -> 55.8 mm
- net Net-(D6-Pad1): track 10.5 -> 6.57 mm
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Other:
- board text added: "OFF"
- board text added: "ON"
