File: Pride Badge.kicad_pcb (KiCad board)
At the start: 2 copper layers, 100 x 130 mm, 93 parts, among them J1 USB_B_Micro, J2 Conn_Batt_JST-PH, J3 SWD_Conn, J4 Conn_SWD20, SW1 PWR_SW, SW2 Mode_BTN, SW3 Bright_BTN, SW4 Reset_BTN, SW5 Boot_SW, SW6 SW_SeeBattGauge, U1 USBLC6-2SC6, U10 555, U2 TP4056, U3 MT3608, U4 AZ1117EH-3.3, U5 FS312F, U6 FS8205, U7 STM32F042F6P6, U8 IS31FL3218, U9 LM339

Commit message: More fixes after prototyping & reading more datasheets
Parts:
- removed R22: 100k, Resistors_SMD:R_0805
- C16: value 4.7n -> 10uF
- R14, R16: value 470R -> 680R
- R15: value 1.1k -> 2k
- R17: value 1k -> 4k3
- R20: value 1k2 -> 680R
- R21: value 900R -> 1k2
- R24: value 700R -> 2k
- R25: value 23k2 -> 27k
- R26: value 34k8 -> 30k
- R27: value 600R -> 3k3
- SW1: footprint my-footprints:Switch_Slide_JS202011SCQN -> digikey-footprints:Switch_Slide_JS202011SCQN
Connections:
- R11 pad 1: Net-(R11-Pad1) -> /Sheet_MCU-LED-Driver/ISSI_SDB
- U1 pad 4: USBDM -> USBDP
- U1 pad 6: USBDP -> USBDM
- U7 pad 17: USBDP -> USBDM
- U7 pad 18: USBDM -> USBDP
- U7 pad 9: (no net) -> /Sheet_MCU-LED-Driver/ISSI_SDB
- U8 pad 24: Net-(R11-Pad1) -> /Sheet_MCU-LED-Driver/ISSI_SDB
Routing:
- net USBDP: track 42.5 -> 47.2 mm, vias 4 -> 6
- net Net-(R11-Pad1): track 2.52 -> 0.00 mm
- net /Sheet_MCU-LED-Driver/ISSI_SDB: track 0.00 -> 2.52 mm
- net /SheetBatteryGauge/LED_VCC: track 54.9 -> 53.0 mm
- net USBDM: track 45.3 -> 44.4 mm, vias 6 -> 4

Commit message: Imported flag shape into outline layer & finished layout
Parts:
- removed J4: Conn_SWD20, Pin_Headers:Pin_Header_Straight_2x10_Pitch2.54mm_SMD
- added C18: 10µF, Capacitors_SMD:C_0805, B.Cu at (133.7, 92.8)
- added D9: LED_Small, LEDs:LED_0805, B.Cu at (70.2, 70.7)
- added Outline_Eco2: pride_badge_outline_100x73, my-footprints:pride_badge_outline_100x73, F.Cu at (112.8, 88.2)
- added R22: 2k7, Resistors_SMD:R_0805, B.Cu at (141.2, 98.2)
- added R28: 2k7, Resistors_SMD:R_0805, B.Cu at (105.2, 68.9)
- added R29: 10k, Resistors_SMD:R_0805, B.Cu at (106.2, 59.0)
- added REF**: 3mm_magnet_hole, my-footprints:3mm_magnet_hole, F.Cu at (111.1, 102.0)
- added REF**: 3mm_magnet_hole, my-footprints:3mm_magnet_hole, F.Cu at (65.9, 65.4)
- added REF**: 3mm_magnet_hole, my-footprints:3mm_magnet_hole, F.Cu at (66.0, 107.7)
- added REF**: 3mm_magnet_hole, my-footprints:3mm_magnet_hole, F.Cu at (159.4, 117.1)
- added REF**: 3mm_magnet_hole, my-footprints:3mm_magnet_hole, F.Cu at (159.7, 74.6)
- added REF**: 3mm_magnet_hole, my-footprints:3mm_magnet_hole, F.Cu at (111.1, 60.3)
- added REF**: HobbyKing 2000mAh JST-PH Cell Outline, my-footprints:HobbyKing 2000mAh JST-PH Cell Outline, F.Cu at (194.2, 44.0)
- added SW7: SW_DPDT_x2, Buttons_Switches_SMD:SW_SPDT_PCM12, B.Cu at (144.7, 96.7)
- added TP1: TP_USBDM, my-footprints:Test_Point_1mm, B.Cu at (140.1, 103.3)
- added TP10: TP_339+_BLUE, my-footprints:Test_Point_1mm, B.Cu at (97.3, 89.1)
- added TP11: TP_339+_GREEN, my-footprints:Test_Point_1mm, B.Cu at (104.1, 87.3)
- added TP12: TP_339+_YELLOW, my-footprints:Test_Point_1mm, B.Cu at (104.0, 85.2)
- added TP13: TP_555THRES, my-footprints:Test_Point_1mm, B.Cu at (86.7, 99.9)
- added TP14: TP_555OUT, my-footprints:Test_Point_1mm, B.Cu at (77.6, 91.2)
- added TP15: TP_339+_ORANGE, my-footprints:Test_Point_1mm, B.Cu at (104.0, 82.5)
- added TP16: TP_339-, my-footprints:Test_Point_1mm, B.Cu at (92.7, 79.2)
- added TP17: TP_MODEBTN, my-footprints:Test_Point_1mm, B.Cu at (90.2, 78.7)
- added TP18: TP_BRIGHTBTN, my-footprints:Test_Point_1mm, B.Cu at (88.3, 77.2)
- added TP19: TP_SWDIO, my-footprints:Test_Point_1mm, B.Cu at (155.2, 75.3)
- added TP2: TP_VUSB, my-footprints:Test_Point_1mm, B.Cu at (152.1, 100.0)
- added TP20: TP_SWCLK, my-footprints:Test_Point_1mm, B.Cu at (143.7, 81.3)
- added TP21: TP_~RST, my-footprints:Test_Point_1mm, B.Cu at (147.7, 81.5)
- added TP22: TP_SDA, my-footprints:Test_Point_1mm, B.Cu at (119.1, 102.9)
- added TP23: TP_SCL, my-footprints:Test_Point_1mm, B.Cu at (114.8, 102.5)
- added TP24: TP_IS_SDB, my-footprints:Test_Point_1mm, B.Cu at (114.0, 79.5)
- added TP25: TP_~RST, my-footprints:Test_Point_1mm, B.Cu at (86.0, 58.7)
- added TP26: TP_BOOT, my-footprints:Test_Point_1mm, B.Cu at (93.7, 61.4)
- added TP27: TP_GND, my-footprints:Test_Point_1mm, B.Cu at (144.6, 106.7)
- added TP28: TP_GND, my-footprints:Test_Point_1mm, B.Cu at (104.7, 94.2)
- added TP29: TP_3V3, my-footprints:Test_Point_1mm, B.Cu at (152.3, 75.3)
- added TP3: TP_5V, my-footprints:Test_Point_1mm, B.Cu at (149.9, 75.3)
- added TP30: TP_555TRIG, my-footprints:Test_Point_1mm, B.Cu at (89.4, 90.3)
- added TP4: TP_3V3, my-footprints:Test_Point_1mm, B.Cu at (153.1, 114.3)
- added TP5: TP_GND, my-footprints:Test_Point_1mm, B.Cu at (150.1, 83.4)
- added TP6: TP_BATT+, my-footprints:Test_Point_1mm, B.Cu at (73.0, 73.7)
- added TP7: TP_BATT-, my-footprints:Test_Point_1mm, B.Cu at (76.9, 73.7)
- added TP8: TP_USBDP, my-footprints:Test_Point_1mm, B.Cu at (142.8, 103.2)
- added TP9: TP_CHRGVCC, my-footprints:Test_Point_1mm, B.Cu at (151.8, 96.7)
- added board_edge_cuts: pride_badge_edge-cuts, my-footprints:pride_badge_edge-cuts, F.Cu at (112.8, 88.2)
- C1: value 10n -> 10nF; moved to B.Cu
- C10: value 4.7uF -> 4.7µF; moved to B.Cu
- C11, C13, C15, C17, C8, C9, D1, D2, D3, D4, D5, D6, D7, D8, F1, J1, L1, R1, R10, R11, R12, R13, R14, R15, R16, R17, R18, R19, R2, R20, R21, R23, R24, R25, R26, R27, R4, R5, R6, R8, R9, SW4, U10, U2, U3, U4, U5, U6, U7, U8, U9: moved to B.Cu
- C12, C14: value 1uF -> 1µF; moved to B.Cu
- C16: value 10uF -> 10µF; moved to B.Cu
- C2: value 100n -> 100nF; moved to B.Cu
- C3: value 4.7u -> 4.7µF; moved to B.Cu
- C4, C5: value 22u -> 22µF; moved to B.Cu
- C6, C7: value 33uF -> 33µF; moved to B.Cu
- J2: value Conn_Batt_JST-PH -> Conn_01x02; footprint Connectors_JST:JST_PH_B2B-PH-SM4-TB_02x2.00mm_Straight -> Connectors_JST:JST_PH_S2B-PH-SM4-TB_02x2.00mm_Angled; moved to B.Cu
- J3: value SWD_Conn -> Custom_SWD; footprint Pin_Headers:Pin_Header_Straight_2x05_Pitch1.27mm_SMD -> w_smd_strip:bb02-hy05a; moved to B.Cu
- L2: value 22uH -> 22µH; moved to B.Cu
- R3: value 1.2k -> 1k2; moved to B.Cu
- R7: value 100 -> 100R; moved to B.Cu
- SW1: value PWR_SW -> SW_DPDT_x2; moved to B.Cu
- SW2, SW3, SW6: footprint my-footprints:Tiny_SMD_Side_Btn_4x2.5mm -> my-footprints:Btn_SMD_6x3.5mm; moved to B.Cu
- SW5: value Boot_SW -> Boot_BTN; footprint Buttons_Switches_SMD:SW_SPDT_PCM12 -> my-footprints:Tiny_SMD_Side_Btn_4x2.5mm; moved to B.Cu
- U1: footprint TO_SOT_Packages_SMD:SOT-23-6 -> digikey-footprints:SOT23-6L; moved to B.Cu
- moved J1 121.8 mm to (159.9, 104.7)
- moved J3 118.9 mm to (158.9, 86.4), turned to 90 degrees
- moved R1 113.0 mm to (155.3, 107.8)
- moved C7 102.1 mm to (151.8, 112.2), turned to 0 degrees
- moved U1 101.6 mm to (148.8, 103.6), turned to 270 degrees
- moved C1 95.9 mm to (147.6, 89.7)
- moved L1 95.6 mm to (149.8, 89.7), turned to 90 degrees
- moved C6 93.3 mm to (147.2, 112.2), turned to 0 degrees
- moved D2 92.8 mm to (159.1, 96.6), turned to 270 degrees
- moved U4 92.5 mm to (148.6, 117.9), turned to 180 degrees
- moved C2 91.3 mm to (145.6, 89.7)
- moved C3 86.5 mm to (143.4, 89.7)
- moved R3 80.2 mm to (141.2, 95.0), turned to 90 degrees
- moved C13 78.3 mm to (114.8, 69.9), turned to 180 degrees
- moved R2 77.1 mm to (139.2, 89.8), turned to 0 degrees
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Connections:
- C8 pad 2: Net-(C8-Pad2) -> -BATT
- J2 pad 1: +BATT -> -BATT
- J2 pad 2: GND -> +BATT
- J3 pad 2: (no net) -> /Sheet_MCU-LED-Driver/SWDIO
- J3 pad 3: GND -> /Sheet_MCU-LED-Driver/SWCLK
- J3 pad 4: (no net) -> /Sheet_MCU-LED-Driver/RESET
- R3 pad 1: Net-(R3-Pad1) -> GND
- R3 pad 2: GND -> Net-(R3-Pad2)
- SW1 pad 1: Net-(F1-Pad2) -> +BATT
- SW1 pad 2: +BATT -> Net-(F1-Pad2)
- SW1 pad 4: (no net) -> +BATT
- SW1 pad 5: (no net) -> Net-(F1-Pad2)
- U2 pad 2: Net-(R3-Pad1) -> Net-(SW7-Pad2)
- U5 pad 6: Net-(C8-Pad2) -> -BATT
- U6 pad 1: Net-(C8-Pad2) -> -BATT
- U7 pad 11: (no net) -> Net-(R28-Pad2)
Routing:
- net +5V: track 308.7 -> 150.9 mm, vias 2 -> 13
- net -BATT: track 0.00 -> 93.0 mm, vias 0 -> 7
- net +3V3: track 232.1 -> 142.4 mm, vias 2 -> 5
- net Net-(DC2-Pad1): track 93.5 -> 10.3 mm, vias 0 -> 1
- net Net-(C4-Pad1): track 15.7 -> 91.3 mm
- net Net-(DD2-Pad1): track 79.8 -> 5.06 mm, vias 0 -> 1
- net Net-(SW3-Pad1): track 11.1 -> 75.0 mm, vias 0 -> 2
- net Net-(SW2-Pad1): track 12.4 -> 69.8 mm, vias 0 -> 2
- net Net-(DE2-Pad1): track 65.8 -> 13.0 mm, vias 0 -> 1
- net Net-(D9-Pad2): track 0.00 -> 41.9 mm, vias 0 -> 4
- net Net-(DD1-Pad1): track 90.6 -> 50.6 mm, vias 0 -> 3
- net Net-(DE1-Pad1): track 76.4 -> 39.2 mm, vias 0 -> 3
- net Net-(R19-Pad2): track 9.97 -> 42.1 mm, vias 0 -> 4
- net Net-(D2-Pad3): track 3.27 -> 34.7 mm
- net +BATT: track 166.4 -> 135.5 mm
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- added copper zone on B.Cu, net GND
Other:
- board size 100 x 130 mm -> 100 x 73.3 mm
- net class Default: clearance 0.3 -> 0.2; via_dia 2 -> 0.8; via_drill 1 -> 0.4
- rule trace_clearance: 0.3 -> 0.2
- rule trace_min: 0.25 -> 0.16
- rule via_min_drill: 0.1 -> 0.3
- rule via_min_size: 0.2 -> 0.16
- board text added: "(Set Charge Current Switch)"
- board text added: "+3V3"
- board text added: "+5V"
- board text added: "+5V 1A"
- board text added: "+BATT"
- board text added: "-BATT"
- board text added: "-Batt+"
- board text added: "0.44A"
- board text added: "1A"
- board text added: "339 -ve"
- board text added: "339+ Blu"
- board text added: "339+ Grn"
- board text added: "339+ Orng"
- board text added: "339+ Yllw"
- board text added: "555 Thres"
- board text added: "555 Trig"
- board text added: "AndrewGillard.com"
- board text added: "BOOT"
- board text added: "BRIGHT"
- board text added: "Batt. Charge Current"
- board text added: "Batt. Level"
- board text added: "Brightness"
- board text added: "Chrg Vcc"
- board text added: "Empty"
- board text added: "Full"
- board text added: "Green: Idle"
- board text added: "Hold to enter bootloader"
- board text added: "ISSI SDB"
- board text added: "Li-Ion/LiPo 500/ 1000mA+ charge current"
- board text added: "MODE"
- board text added: "POWER"
- board text added: "Pride Badge r1 2018-07"
- board text added: "RESET"
- board text added: "Red: Charge"
- board text added: "SCL"
- board text added: "SDA"
- board text added: "SWCLK"
- board text added: "SWD"
- board text added: "SWDIO"
- board text added: "Show Batt. Level"
- board text added: "USB D+"
- board text added: "USB D-"
- board text added: "VUSB"
- board text added: "V_LED"
- board text added: "~RST"
- board text removed: "- Batt +"
- board text removed: "1"
- board text removed: "3V3"
- board text removed: "5V"
- board text removed: "Bootloader"
- board text removed: "Bright"
- board text removed: "D+"
- board text removed: "D-"
- board text removed: "Normal"
- board text removed: "SC"
- board text removed: "SD"
- board text removed: "Show Batt Level"
- board text removed: "USB"
- board text removed: "Vbatt"
