File: power.sch (KiCad schematic (older format))
At the start: 23 parts

Commit message: Schematics complete, ready for prototype PCBs to be designed
Parts:
- removed C?: 10u, symbol Device:C
- added C1: 10n, Capacitors_SMD:C_0805, symbol Device:C
- added C2: 100n, Capacitors_SMD:C_0805, symbol Device:C
- added C3: 4.7u, Capacitors_SMD:C_0805, symbol Device:C
- added C6, C7: 33uF, Capacitors_SMD:C_0805, symbol Device:C
- added L1: L, w_smd_inductors:inductor_smd_0805, symbol Device:L
- added R1: 100k, Resistors_SMD:R_0805, symbol Device:R
- added U1: USBLC6-2SC6, Package_TO_SOT_SMD:SOT-23-6, symbol Power_Protection:USBLC6-2SC6
- C4, C5, C8: renamed from C?; footprint (none) -> Capacitors_SMD:C_0805
- D1: renamed from D?; footprint (none) -> Diodes_SMD:D_SMA
- D2: renamed from D?; footprint (none) -> LEDs:LED_0606
- F1: renamed from F?; footprint (none) -> Fuse_Holders_and_Fuses:Fuse_SMD1206_Reflow
- J1: renamed from J?; footprint (none) -> my-footprints:USB_Micro-B_OSHPark
- J2: renamed from J?; footprint (none) -> Connectors_JST:JST_PH_B2B-PH-SM4-TB_02x2.00mm_Straight
- L2: renamed from L?; footprint (none) -> Inductors:Inductor_Wurth_HCM-7070
- R2, R3, R4, R5, R6, R7, R8: renamed from R?; footprint (none) -> Resistors_SMD:R_0805
- SW1: renamed from SW?; footprint (none) -> digikey-footprints:Switch_Slide_JS202011SCQN
- U2: renamed from U?; footprint (none) -> SMD_Packages:SOIC-8-N
- U3, U5, U6: renamed from U?; footprint (none) -> TO_SOT_Packages_SMD:SOT-23-6
- gave numbers to parts that had none: 1
Connections:
- wire segments 67 -> 92
- no-connect marks 2 -> 1

Commit message: Fix footprint of dual 0603 LED
Parts:
- D2: footprint LEDs:LED_0606 -> my-footprints:LED_0606 (Dual - 0603x2)
- U4: symbol dk_PMIC-Voltage-Regulators-Linear:NCP1117ST33T3G -> Pride-Badge-rescue:NCP1117ST33T3G-dk_PMIC-Voltage-Regulators-Linear
Changed lines of the file:
@@
 F 0 "D2" V 2696 4738 50  0000 L CNN
 F 1 "LED_GREEN1_RED2" V 2605 4738 50  0000 L CNN
-F 2 "LEDs:LED_0606" H 2680 4450 50  0001 C CNN
+F 2 "my-footprints:LED_0606 (Dual - 0603x2)" H 2680 4450 50  0001 C CNN
 F 3 "~" H 2680 4450 50  0001 C CNN
 	1    2650 4450
@@
 $EndComp
 $Comp
-L dk_PMIC-Voltage-Regulators-Linear:NCP1117ST33T3G U4
+L Pride-Badge-rescue:NCP1117ST33T3G-dk_PMIC-Voltage-Regulators-Linear U4
 U 1 1 5B35A4A8
 P 8900 5350

Commit message: Prototype PCB laid out, no tracks yet
Parts:
- U1: footprint Package_TO_SOT_SMD:SOT-23-6 -> TO_SOT_Packages_SMD:SOT-23-6
- U2: footprint SMD_Packages:SOIC-8-N -> digikey-footprints:SOIC-8-1EP_W3.9mm
Changed lines of the file:
@@
 F 0 "U2" H 3500 3765 50  0000 C CNN
 F 1 "TP4056" H 3500 3674 50  0000 C CNN
-F 2 "SMD_Packages:SOIC-8-N" H 3500 3300 50  0001 C CNN
+F 2 "digikey-footprints:SOIC-8-1EP_W3.9mm" H 3500 3300 50  0001 C CNN
 F 3 "" H 3500 3300 50  0001 C CNN
 	1    3500 3300
@@
 F 0 "U1" V 2000 1400 50  0000 R CNN
 F 1 "USBLC6-2SC6" V 2700 1450 50  0000 R CNN
-F 2 "Package_TO_SOT_SMD:SOT-23-6" H 1600 2000 50  0001 C CNN
+F 2 "TO_SOT_Packages_SMD:SOT-23-6" H 1600 2000 50  0001 C CNN
 F 3 "http://www2.st.com/resource/en/datasheet/CD00050750.pdf" H 2550 1950 50  0001 C CNN
 	1    2350 1600

Commit message: Prototype PCB design finished?
Parts:
- U1: symbol Power_Protection:USBLC6-2SC6 -> dk_TVS-Diodes:USBLC6-2SC6
Connections:
- net labels added: USBDM, USBDP
- net labels removed: USB_D+, USB_D-
- wire segments 92 -> 93
Changed lines of the file:
@@
 	900  1950 850  1950
 Connection ~ 850  1950
-Text HLabel 2250 1100 1    50   Input ~ 0
-USB_D+
-Text HLabel 2250 2100 3    50   Input ~ 0
-USB_D-
 Text HLabel 1250 1350 1    50   Input ~ 0
 VUSB
@@
 Wire Wire Line
 	2550 4750 2750 4750
-Text HLabel 2650 4750 3    50   Input ~ 0
-VUSB
 Wire Wire Line
 	3500 4100 3550 4100
@@
 	9500 5750 8800 5750
 $Comp
-L Power_Protection:USBLC6-2SC6 U1
+L dk_TVS-Diodes:USBLC6-2SC6 U1
 U 1 1 5B469059
-P 2350 1600
-F 0 "U1" V 2000 1400 50  0000 R CNN
-F 1 "USBLC6-2SC6" V 2700 1450 50  0000 R CNN
-F 2 "TO_SOT_Packages_SMD:SOT-23-6" H 1600 2000 50  0001 C CNN
-F 3 "http://www2.st.com/resource/en/datasheet/CD00050750.pdf" H 2550 1950 50  0001 C CNN
-	1    2350 1600
-	0    -1   -1   0
-$EndComp
-Wire Wire Line
-	1850 1600 1850 1350
-Wire Wire Line
-	1850 1350 1200 1350
+P 2400 1650
+F 0 "U1" H 2800 2200 50  0000 R CNN
+F 1 "USBLC6-2SC6" H 2550 2200 50  0000 R CNN
+F 2 "TO_SOT_Packages_SMD:SOT-23-6" H 1650 2050 50  0001 C CNN
+F 3 "http://www2.st.com/resource/en/datasheet/CD00050750.pdf" H 2600 2000 50  0001 C CNN
+	1    2400 1650
+	1    0    0    -1
+$EndComp
 $Comp
 L power:GND #PWR0123
 U 1 1 5B46C80F
-P 2850 1700
-F 0 "#PWR0123" H 2850 1450 50  0001 C CNN
-F 1 "GND" H 2855 1527 50  0000 C CNN
-F 2 "" H 2850 1700 50  0001 C CNN
-F 3 "" H 2850 1700 50  0001 C CNN
-	1    2850 1700
-	1    0    0    -1
-$EndComp
-Wire Wire Line
-	2850 1700 2850 1600
-Wire Wire Line
-	1200 1650 1600 1650
-Wire Wire Line
-	1600 1650 1600 2100
-Wire Wire Line
-	1600 2100 2050 2100
-Wire Wire Line
-	2050 2100 2050 2600
-Wire Wire Line
-	2050 2600 2450 2600
-Wire Wire Line
-	2450 2600 2450 2100
+P 1850 1650
+F 0 "#PWR0123" H 1850 1400 50  0001 C CNN
+F 1 "GND" H 1855 1477 50  0000 C CNN
+F 2 "" H 1850 1650 50  0001 C CNN
+F 3 "" H 1850 1650 50  0001 C CNN
+	1    1850 1650
+	1    0    0    -1
+$EndComp
 Wire Wire Line
 	1200 1550 1600 1550
-Wire Wire Line
-	1600 1550 1600 1050
-Wire Wire Line
-	1600 1050 2100 1050
-Wire Wire Line
-	2100 1050 2100 600
-Wire Wire Line
-	2100 600  2450 600
-Wire Wire Line
-	2450 600  2450 1100
 $Comp
 L Device:R R1
@@
 Connection ~ 1800 3400
 Wire Wire Line
-	2250 3100 2850 3100
+	2250 3100 2650 3100
 Connection ~ 2250 3100
 Connection ~ 2050 3400
 Wire Wire Line
 	2050 3400 1800 3400
+Wire Wire Line
+	1900 1650 1850 1650
+Wire Wire Line
+	1250 1350 1200 1350
+Text HLabel 3000 1650 2    50   Input ~ 0
+VUSB
+Wire Wire Line
+	2900 1650 3000 1650
+Wire Wire Line
+	2900 1350 3000 1350
+Wire Wire Line
+	2900 1950 3000 1950
+Wire Wire Line
+	1750 1650 1750 1350
+Wire Wire Line
+	1750 1350 1900 1350
+Wire Wire Line
+	1200 1650 1750 1650
+Wire Wire Line
+	1600 1550 1600 1950
+Wire Wire Line
+	1600 1950 1900 1950
+Text GLabel 3000 1350 2    50   BiDi ~ 0
+USBDP
+Text GLabel 3000 1950 2    50   BiDi ~ 0
+USBDM
+Wire Wire Line
+	2550 4750 2400 4750
+Wire Wire Line
+	2400 4750 2400 3400
+Wire Wire Line
+	2400 3400 2650 3400
+Wire Wire Line
+	2650 3400 2650 3100
+Connection ~ 2550 4750
+Connection ~ 2650 3100
+Wire Wire Line
+	2650 3100 2850 3100
 $EndSCHEMATC

Commit message: Fixed up PCB design after fixing some IC footprints
Parts:
- SW1: footprint digikey-footprints:Switch_Slide_JS202011SCQN -> my-footprints:Switch_Slide_JS202011SCQN
Changed lines of the file:
@@
 F 0 "SW1" H 7400 4035 50  0000 C CNN
 F 1 "PWR_SW" H 7400 3944 50  0000 C CNN
-F 2 "digikey-footprints:Switch_Slide_JS202011SCQN" H 7400 3750 50  0001 C CNN
+F 2 "my-footprints:Switch_Slide_JS202011SCQN" H 7400 3750 50  0001 C CNN
 F 3 "" H 7400 3750 50  0001 C CNN
 	1    7400 3750

Commit message: More fixes after testing the LED gauge and such
Parts:
- SW1: footprint my-footprints:Switch_Slide_JS202011SCQN -> digikey-footprints:Switch_Slide_JS202011SCQN
Changed lines of the file:
@@
 	2850 3100 3000 3100
 Wire Wire Line
-	4000 3450 4200 3450
+	4000 3450 4050 3450
 Wire Wire Line
 	4200 3450 4200 3500
@@
 F 0 "SW1" H 7400 4035 50  0000 C CNN
 F 1 "PWR_SW" H 7400 3944 50  0000 C CNN
-F 2 "my-footprints:Switch_Slide_JS202011SCQN" H 7400 3750 50  0001 C CNN
+F 2 "digikey-footprints:Switch_Slide_JS202011SCQN" H 7400 3750 50  0001 C CNN
 F 3 "" H 7400 3750 50  0001 C CNN
 	1    7400 3750
@@
 $EndComp
 Wire Wire Line
-	4000 3100 4100 3100
+	4000 3100 4050 3100
 $Comp
 L Device:C C8

Commit message: More fixes after prototyping & reading more datasheets
Parts:
- removed J2: Conn_Batt_JST-PH, Connectors_JST:JST_PH_B2B-PH-SM4-TB_02x2.00mm_Straight, symbol Connector_Generic:Conn_01x02
- added C?: 10u, Capacitors_SMD:C_0805, symbol Device:C
- added J?: Conn_01x02, Connectors_JST:JST_PH_S2B-PH-SM4-TB_02x2.00mm_Angled, symbol Connector_Generic:Conn_01x02
- U1: footprint TO_SOT_Packages_SMD:SOT-23-6 -> digikey-footprints:SOT23-6L
Connections:
- net labels added: -BATT
- wire segments 93 -> 97
Changed lines of the file:
@@
 Wire Wire Line
 	8450 4300 8450 4200
-$Comp
-L Connector_Generic:Conn_01x02 J2
-U 1 1 5B35AB89
-P 6050 2050
-F 0 "J2" H 5970 2267 50  0000 C CNN
-F 1 "Conn_Batt_JST-PH" H 6200 2150 50  0000 C CNN
-F 2 "Connectors_JST:JST_PH_B2B-PH-SM4-TB_02x2.00mm_Straight" H 6050 2050 50  0001 C CNN
-F 3 "~" H 6050 2050 50  0001 C CNN
-	1    6050 2050
-	-1   0    0    -1
-$EndComp
-$Comp
-L power:GND #PWR0112
-U 1 1 5B35AE38
-P 6550 2150
-F 0 "#PWR0112" H 6550 1900 50  0001 C CNN
-F 1 "GND" H 6555 1977 50  0000 C CNN
-F 2 "" H 6550 2150 50  0001 C CNN
-F 3 "" H 6550 2150 50  0001 C CNN
-	1    6550 2150
-	1    0    0    -1
-$EndComp
-Wire Wire Line
-	6550 2150 6250 2150
-Wire Wire Line
-	6250 2050 6550 2050
-Text HLabel 4450 800  3    50   Input ~ 0
+Text HLabel 4450 700  3    50   Input ~ 0
 VBATT
-$Comp
-L power:+BATT #PWR0113
-U 1 1 5B35ADD9
-P 6550 2050
-F 0 "#PWR0113" H 6550 1900 50  0001 C CNN
-F 1 "+BATT" H 6565 2223 50  0000 C CNN
-F 2 "" H 6550 2050 50  0001 C CNN
-F 3 "" H 6550 2050 50  0001 C CNN
-	1    6550 2050
-	1    0    0    -1
-$EndComp
 $Comp
 L power:+BATT #PWR0114
@@
 L power:+BATT #PWR0116
 U 1 1 5B35DF99
-P 4450 800
-F 0 "#PWR0116" H 4450 650 50  0001 C CNN
-F 1 "+BATT" H 4465 973 50  0000 C CNN
-F 2 "" H 4450 800 50  0001 C CNN
-F 3 "" H 4450 800 50  0001 C CNN
-	1    4450 800
+P 4450 700
+F 0 "#PWR0116" H 4450 550 50  0001 C CNN
+F 1 "+BATT" H 4465 873 50  0000 C CNN
+F 2 "" H 4450 700 50  0001 C CNN
+F 3 "" H 4450 700 50  0001 C CNN
+	1    4450 700
 	1    0    0    -1
 $EndComp
@@
 L power:GND #PWR0117
 U 1 1 5B35E00F
-P 5000 900
-F 0 "#PWR0117" H 5000 650 50  0001 C CNN
-F 1 "GND" H 5005 727 50  0000 C CNN
-F 2 "" H 5000 900 50  0001 C CNN
-F 3 "" H 5000 900 50  0001 C CNN
-	1    5000 900
-	1    0    0    -1
-$EndComp
-Text HLabel 5000 900  1    50   Input ~ 0
+P 5000 800
+F 0 "#PWR0117" H 5000 550 50  0001 C CNN
+F 1 "GND" H 5005 627 50  0000 C CNN
+F 2 "" H 5000 800 50  0001 C CNN
+F 3 "" H 5000 800 50  0001 C CNN
+	1    5000 800
+	1    0    0    -1
+$EndComp
+Text HLabel 5000 800  1    50   Input ~ 0
 GND
 $Comp
 L power:+5V #PWR0118
 U 1 1 5B35E570
-P 5550 850
-F 0 "#PWR0118" H 5550 700 50  0001 C CNN
-F 1 "+5V" H 5565 1023 50  0000 C CNN
-F 2 "" H 5550 850 50  0001 C CNN
-F 3 "" H 5550 850 50  0001 C CNN
-	1    5550 850
-	1    0    0    -1
-$EndComp
-Text HLabel 5550 850  3    50   Input ~ 0
+P 5550 750
+F 0 "#PWR0118" H 5550 600 50  0001 C CNN
+F 1 "+5V" H 5565 923 50  0000 C CNN
+F 2 "" H 5550 750 50  0001 C CNN
+F 3 "" H 5550 750 50  0001 C CNN
+	1    5550 750
+	1    0    0    -1
+$EndComp
+Text HLabel 5550 750  3    50   Input ~ 0
 5V
 $Comp
@@
 L power:+3.3V #PWR0121
 U 1 1 5B35A764
-P 6000 850
-F 0 "#PWR0121" H 6000 700 50  0001 C CNN
-F 1 "+3.3V" H 6015 1023 50  0000 C CNN
-F 2 "" H 6000 850 50  0001 C CNN
-F 3 "" H 6000 850 50  0001 C CNN
-	1    6000 850
-	1    0    0    -1
-$EndComp
-Text HLabel 6000 850  3    50   Input ~ 0
+P 6000 750
+F 0 "#PWR0121" H 6000 600 50  0001 C CNN
+F 1 "+3.3V" H 6015 923 50  0000 C CNN
+F 2 "" H 6000 750 50  0001 C CNN
+F 3 "" H 6000 750 50  0001 C CNN
+	1    6000 750
+	1    0    0    -1
+$EndComp
+Text HLabel 6000 750  3    50   Input ~ 0
 3V3
 $Comp
@@
 F 0 "U1" H 2800 2200 50  0000 R CNN
 F 1 "USBLC6-2SC6" H 2550 2200 50  0000 R CNN
-F 2 "TO_SOT_Packages_SMD:SOT-23-6" H 1650 2050 50  0001 C CNN
+F 2 "digikey-footprints:SOT23-6L" H 1650 2050 50  0001 C CNN
 F 3 "http://www2.st.com/resource/en/datasheet/CD00050750.pdf" H 2600 2000 50  0001 C CNN
 	1    2400 1650
@@
 Wire Wire Line
 	1600 1950 1900 1950
+Text GLabel 3000 1950 2    50   BiDi ~ 0
+USBDP
 Text GLabel 3000 1350 2    50   BiDi ~ 0
-USBDP
-Text GLabel 3000 1950 2    50   BiDi ~ 0
 USBDM
 Wire Wire Line
@@
 Wire Wire Line
 	2650 3100 2850 3100
+Wire Wire Line
+	5450 3700 5700 3700
+$Comp
+L Connector_Generic:Conn_01x02 J?
+U 1 1 5B44F270
+P 5250 3700
+F 0 "J?" H 5170 3375 50  0000 C CNN
+F 1 "Conn_01x02" H 5170 3466 50  0000 C CNN
+F 2 "Connectors_JST:JST_PH_S2B-PH-SM4-TB_02x2.00mm_Angled" H 5250 3700 50  0001 C CNN
+F 3 "~" H 5250 3700 50  0001 C CNN
+	1    5250 3700
+	-1   0    0    1
+$EndComp
+$Comp
+L power:+BATT #PWR?
+U 1 1 5B4607AE
+P 5700 3600
+F 0 "#PWR?" H 5700 3450 50  0001 C CNN
+F 1 "+BATT" H 5715 3773 50  0000 C CNN
+F 2 "" H 5700 3600 50  0001 C CNN
+F 3 "" H 5700 3600 50  0001 C CNN
+	1    5700 3600
+	1    0    0    -1
+$EndComp
+Wire Wire Line
+	5450 3600 5700 3600
+$Comp
+L power:-BATT #PWR?
+U 1 1 5B47C670
+P 5700 3700
+F 0 "#PWR?" H 5700 3550 50  0001 C CNN
+F 1 "-BATT" H 5715 3873 50  0000 C CNN
+F 2 "" H 5700 3700 50  0001 C CNN
+F 3 "" H 5700 3700 50  0001 C CNN
+	1    5700 3700
+	-1   0    0    1
+$EndComp
+$Comp
+L power:-BATT #PWR?
+U 1 1 5B47C7B9
+P 4450 5950
+F 0 "#PWR?" H 4450 5800 50  0001 C CNN
+F 1 "-BATT" H 4465 6123 50  0000 C CNN
+F 2 "" H 4450 5950 50  0001 C CNN
+F 3 "" H 4450 5950 50  0001 C CNN
+	1    4450 5950
+	-1   0    0    1
+$EndComp
+Wire Wire Line
+	4450 5950 4800 5950
+$Comp
+L Device:C C?
+U 1 1 5B48173E
+P 4050 3250
+F 0 "C?" H 4165 3296 50  0000 L CNN
+F 1 "10u" H 4165 3205 50  0000 L CNN
+F 2 "Capacitors_SMD:C_0805" H 4088 3100 50  0001 C CNN
+F 3 "~" H 4050 3250 50  0001 C CNN
+	1    4050 3250
+	1    0    0    -1
+$EndComp
+Connection ~ 4050 3100
+Wire Wire Line
+	4050 3100 4100 3100
+Wire Wire Line
+	4050 3400 4050 3450
+Connection ~ 4050 3450
+Wire Wire Line
+	4050 3450 4200 3450
 $EndSCHEMATC

Commit message: Hopefully final schematic fixes
Parts:
- gave numbers to parts that had none: 2
Changed lines of the file:
@@
 	5450 3700 5700 3700
 $Comp
-L Connector_Generic:Conn_01x02 J?
+L Connector_Generic:Conn_01x02 J2
 U 1 1 5B44F270
 P 5250 3700
-F 0 "J?" H 5170 3375 50  0000 C CNN
+F 0 "J2" H 5170 3375 50  0000 C CNN
 F 1 "Conn_01x02" H 5170 3466 50  0000 C CNN
 F 2 "Connectors_JST:JST_PH_S2B-PH-SM4-TB_02x2.00mm_Angled" H 5250 3700 50  0001 C CNN
@@
 $EndComp
 $Comp
-L power:+BATT #PWR?
+L power:+BATT #PWR0112
 U 1 1 5B4607AE
 P 5700 3600
-F 0 "#PWR?" H 5700 3450 50  0001 C CNN
+F 0 "#PWR0112" H 5700 3450 50  0001 C CNN
 F 1 "+BATT" H 5715 3773 50  0000 C CNN
 F 2 "" H 5700 3600 50  0001 C CNN
@@
 	5450 3600 5700 3600
 $Comp
-L power:-BATT #PWR?
+L power:-BATT #PWR0113
 U 1 1 5B47C670
 P 5700 3700
-F 0 "#PWR?" H 5700 3550 50  0001 C CNN
+F 0 "#PWR0113" H 5700 3550 50  0001 C CNN
 F 1 "-BATT" H 5715 3873 50  0000 C CNN
 F 2 "" H 5700 3700 50  0001 C CNN
@@
 $EndComp
 $Comp
-L power:-BATT #PWR?
+L power:-BATT #PWR0131
 U 1 1 5B47C7B9
 P 4450 5950
-F 0 "#PWR?" H 4450 5800 50  0001 C CNN
+F 0 "#PWR0131" H 4450 5800 50  0001 C CNN
 F 1 "-BATT" H 4465 6123 50  0000 C CNN
 F 2 "" H 4450 5950 50  0001 C CNN
@@
 	4450 5950 4800 5950
 $Comp
-L Device:C C?
+L Device:C C18
 U 1 1 5B48173E
 P 4050 3250
-F 0 "C?" H 4165 3296 50  0000 L CNN
+F 0 "C18" H 4165 3296 50  0000 L CNN
 F 1 "10u" H 4165 3205 50  0000 L CNN
 F 2 "Capacitors_SMD:C_0805" H 4088 3100 50  0001 C CNN
