File: power.sch (KiCad schematic (older format))
At the start: 31 parts, among them J1 USB_B_Micro, J2 Conn_01x02, SW1 PWR_SW, U1 USBLC6-2SC6, U2 TP4056, U3 MT3608, U4 AZ1117EH-3.3, U5 FS312F, U6 FS8205

Commit message: Imported flag shape into outline layer & finished layout
Parts:
- added R22: 2k7, Resistors_SMD:R_0805, symbol Device:R
- added unit 2 of SW1
- added SW7: SW_DPDT_x2, Buttons_Switches_SMD:SW_SPDT_PCM12, symbol Switch:SW_DPDT_x2
- added TP1: TP_USBDM, my-footprints:Test_Point_1mm, symbol Connector_Specialized:Test_Point
- added TP2: TP_VUSB, my-footprints:Test_Point_1mm, symbol Connector_Specialized:Test_Point
- added TP3: TP_5V, my-footprints:Test_Point_1mm, symbol Connector_Specialized:Test_Point
- added TP4: TP_3V3, my-footprints:Test_Point_1mm, symbol Connector_Specialized:Test_Point
- added TP5: TP_GND, my-footprints:Test_Point_1mm, symbol Connector_Specialized:Test_Point
- added TP6: TP_BATT+, my-footprints:Test_Point_1mm, symbol Connector_Specialized:Test_Point
- added TP7: TP_BATT-, my-footprints:Test_Point_1mm, symbol Connector_Specialized:Test_Point
- added TP8: TP_USBDP, my-footprints:Test_Point_1mm, symbol Connector_Specialized:Test_Point
- added TP9: TP_CHRGVCC, my-footprints:Test_Point_1mm, symbol Connector_Specialized:Test_Point
- C1: value 10n -> 10nF
- C18: value 10u -> 10µF
- C2: value 100n -> 100nF
- C3: value 4.7u -> 4.7µF
- C4, C5: value 22u -> 22µF
- C6, C7: value 33uF -> 33µF
- L2: value 22uH -> 22µH
- R3: value 1.2k -> 1k2
- R7: value 100 -> 100R
- SW1: value PWR_SW -> SW_DPDT_x2
Connections:
- wire segments 97 -> 111
- no-connect marks 1 -> 3
Other:
- note added: "Charge current selection.\n1k2 = 1A\n2k7 = 444mA"
