File: BatteryGauge.sch (KiCad schematic (older format))
At the start: 29 parts

Commit message: Schematics complete, ready for prototype PCBs to be designed
Parts:
- C16, C17: renamed from C?; footprint (none) -> Capacitors_SMD:C_0805
- D3: renamed from D?; footprint (none) -> Diodes_SMD:D_MiniMELF_Handsoldering
- D4, D5, D6, D7, D8: renamed from D?; footprint (none) -> Diodes_SMD:D_0805
- R13, R14, R15, R16, R17, R18, R19, R20, R21, R22, R23, R24, R25, R26, R27: renamed from R?; footprint (none) -> Resistors_SMD:R_0805
- SW6: renamed from SW?; footprint (none) -> my-footprints:Tiny_SMD_Side_Btn_4x2.5mm
- U10: renamed from U?; footprint (none) -> digikey-footprints:SOIC-8_W3.9mm
- U9: renamed from U?; footprint (none) -> digikey-footprints:SOIC-24_W7.50mm

Commit message: Prototype PCB laid out, no tracks yet
Parts:
- R14, R16: value R -> 470R
- R20: value R -> 1k2
- R23: value R -> 8k66
- R25: value R -> 23k2
- R26: value R -> 34k8
Changed lines of the file:
@@
 P 7150 5400
 F 0 "R26" H 7220 5446 50  0000 L CNN
-F 1 "R" H 7220 5355 50  0000 L CNN
+F 1 "34k8" H 7220 5355 50  0000 L CNN
 F 2 "Resistors_SMD:R_0805" V 7080 5400 50  0001 C CNN
 F 3 "~" H 7150 5400 50  0001 C CNN
@@
 P 6700 4750
 F 0 "R23" H 6770 4796 50  0000 L CNN
-F 1 "R" H 6770 4705 50  0000 L CNN
+F 1 "8k66" H 6770 4705 50  0000 L CNN
 F 2 "Resistors_SMD:R_0805" V 6630 4750 50  0001 C CNN
 F 3 "~" H 6700 4750 50  0001 C CNN
@@
 P 6700 2350
 F 0 "R14" H 6770 2396 50  0000 L CNN
-F 1 "R" H 6770 2305 50  0000 L CNN
+F 1 "470R" H 6770 2305 50  0000 L CNN
 F 2 "Resistors_SMD:R_0805" V 6630 2350 50  0001 C CNN
 F 3 "~" H 6700 2350 50  0001 C CNN
@@
 P 6700 3200
 F 0 "R16" H 6770 3246 50  0000 L CNN
-F 1 "R" H 6770 3155 50  0000 L CNN
+F 1 "470R" H 6770 3155 50  0000 L CNN
 F 2 "Resistors_SMD:R_0805" V 6630 3200 50  0001 C CNN
 F 3 "~" H 6700 3200 50  0001 C CNN
@@
 P 6700 3950
 F 0 "R20" H 6770 3996 50  0000 L CNN
-F 1 "R" H 6770 3905 50  0000 L CNN
+F 1 "1k2" H 6770 3905 50  0000 L CNN
 F 2 "Resistors_SMD:R_0805" V 6630 3950 50  0001 C CNN
 F 3 "~" H 6700 3950 50  0001 C CNN
@@
 P 7150 4950
 F 0 "R25" H 7220 4996 50  0000 L CNN
-F 1 "R" H 7220 4905 50  0000 L CNN
+F 1 "23k2" H 7220 4905 50  0000 L CNN
 F 2 "Resistors_SMD:R_0805" V 7080 4950 50  0001 C CNN
 F 3 "~" H 7150 4950 50  0001 C CNN

Commit message: Fixed footprints for a few ICs. Oops.
Updated PCB layout to come!
Parts:
- U9: footprint digikey-footprints:SOIC-24_W7.50mm -> digikey-footprints:SOIC-14_W3.9mm
Changed lines of the file:
@@
 F 0 "U9" H 8191 3246 50  0000 L CNN
 F 1 "LM339" H 8191 3155 50  0000 L CNN
-F 2 "digikey-footprints:SOIC-24_W7.50mm" H 7800 3300 50  0001 C CNN
+F 2 "digikey-footprints:SOIC-14_W3.9mm" H 7800 3300 50  0001 C CNN
 F 3 "http://www.ti.com/lit/ds/symlink/lm339.pdf" H 7900 3400 50  0001 C CNN
 	2    7850 3200

Commit message: Fixed up PCB design after fixing some IC footprints
Parts:
- U9: footprint digikey-footprints:SOIC-24_W7.50mm -> digikey-footprints:SOIC-14_W3.9mm
Changed lines of the file:
@@
 F 0 "U9" H 7991 2446 50  0000 L CNN
 F 1 "LM339" H 7991 2355 50  0000 L CNN
-F 2 "digikey-footprints:SOIC-24_W7.50mm" H 7600 2500 50  0001 C CNN
+F 2 "digikey-footprints:SOIC-14_W3.9mm" H 7600 2500 50  0001 C CNN
 F 3 "http://www.ti.com/lit/ds/symlink/lm339.pdf" H 7700 2600 50  0001 C CNN
 	1    7650 2400
@@
 F 0 "U9" H 8391 3996 50  0000 L CNN
 F 1 "LM339" H 8391 3905 50  0000 L CNN
-F 2 "digikey-footprints:SOIC-24_W7.50mm" H 8000 4050 50  0001 C CNN
+F 2 "digikey-footprints:SOIC-14_W3.9mm" H 8000 4050 50  0001 C CNN
 F 3 "http://www.ti.com/lit/ds/symlink/lm339.pdf" H 8100 4150 50  0001 C CNN
 	3    8050 3950
@@
 F 0 "U9" H 8641 4796 50  0000 L CNN
 F 1 "LM339" H 8641 4705 50  0000 L CNN
-F 2 "digikey-footprints:SOIC-24_W7.50mm" H 8250 4850 50  0001 C CNN
+F 2 "digikey-footprints:SOIC-14_W3.9mm" H 8250 4850 50  0001 C CNN
 F 3 "http://www.ti.com/lit/ds/symlink/lm339.pdf" H 8350 4950 50  0001 C CNN
 	4    8300 4750

Commit message: More fixes after testing the LED gauge and such
Parts:
- removed R22: 100k, Resistors_SMD:R_0805, symbol Device:R
- C16: value 4.7n -> 10uF
- R14, R16: value 470R -> 680R
- R15: value 1.1k -> 2k
- R17: value 1k -> 4k3
- R20: value 1k2 -> 680R
- R21: value 900R -> 1k2
- R24: value 700R -> 2k
- R25: value 23k2 -> 27k
- R26: value 34k8 -> 30k
- R27: value 600R -> 3k3
Connections:
- wire segments 91 -> 87
Other:
- note added: "~~1.95V here"
Changed lines of the file:
@@
 P 7150 5400
 F 0 "R26" H 7220 5446 50  0000 L CNN
-F 1 "34k8" H 7220 5355 50  0000 L CNN
+F 1 "30k" H 7220 5355 50  0000 L CNN
 F 2 "Resistors_SMD:R_0805" V 7080 5400 50  0001 C CNN
 F 3 "~" H 7150 5400 50  0001 C CNN
@@
 P 9500 2400
 F 0 "R15" V 9293 2400 50  0000 C CNN
-F 1 "1.1k" V 9384 2400 50  0000 C CNN
+F 1 "2k" V 9384 2400 50  0000 C CNN
 F 2 "Resistors_SMD:R_0805" V 9430 2400 50  0001 C CNN
 F 3 "~" H 9500 2400 50  0001 C CNN
@@
 P 9500 3200
 F 0 "R17" V 9293 3200 50  0000 C CNN
-F 1 "1k" V 9384 3200 50  0000 C CNN
+F 1 "4k3" V 9384 3200 50  0000 C CNN
 F 2 "Resistors_SMD:R_0805" V 9430 3200 50  0001 C CNN
 F 3 "~" H 9500 3200 50  0001 C CNN
@@
 P 9500 3950
 F 0 "R21" V 9293 3950 50  0000 C CNN
-F 1 "900R" V 9384 3950 50  0000 C CNN
+F 1 "1k2" V 9384 3950 50  0000 C CNN
 F 2 "Resistors_SMD:R_0805" V 9430 3950 50  0001 C CNN
 F 3 "~" H 9500 3950 50  0001 C CNN
@@
 P 9500 4750
 F 0 "R24" V 9293 4750 50  0000 C CNN
-F 1 "700R" V 9384 4750 50  0000 C CNN
+F 1 "2k" V 9384 4750 50  0000 C CNN
 F 2 "Resistors_SMD:R_0805" V 9430 4750 50  0001 C CNN
 F 3 "~" H 9500 4750 50  0001 C CNN
@@
 P 9500 5400
 F 0 "R27" V 9293 5400 50  0000 C CNN
-F 1 "600R" V 9384 5400 50  0000 C CNN
+F 1 "3k3" V 9384 5400 50  0000 C CNN
 F 2 "Resistors_SMD:R_0805" V 9430 5400 50  0001 C CNN
 F 3 "~" H 9500 5400 50  0001 C CNN
@@
 P 6700 2350
 F 0 "R14" H 6770 2396 50  0000 L CNN
-F 1 "470R" H 6770 2305 50  0000 L CNN
+F 1 "680R" H 6770 2305 50  0000 L CNN
 F 2 "Resistors_SMD:R_0805" V 6630 2350 50  0001 C CNN
 F 3 "~" H 6700 2350 50  0001 C CNN
@@
 P 6700 3200
 F 0 "R16" H 6770 3246 50  0000 L CNN
-F 1 "470R" H 6770 3155 50  0000 L CNN
+F 1 "680R" H 6770 3155 50  0000 L CNN
 F 2 "Resistors_SMD:R_0805" V 6630 3200 50  0001 C CNN
 F 3 "~" H 6700 3200 50  0001 C CNN
@@
 P 6700 3950
 F 0 "R20" H 6770 3996 50  0000 L CNN
-F 1 "1k2" H 6770 3905 50  0000 L CNN
+F 1 "680R" H 6770 3905 50  0000 L CNN
 F 2 "Resistors_SMD:R_0805" V 6630 3950 50  0001 C CNN
 F 3 "~" H 6700 3950 50  0001 C CNN
@@
 P 7150 4950
 F 0 "R25" H 7220 4996 50  0000 L CNN
-F 1 "23k2" H 7220 4905 50  0000 L CNN
+F 1 "27k" H 7220 4905 50  0000 L CNN
 F 2 "Resistors_SMD:R_0805" V 7080 4950 50  0001 C CNN
 F 3 "~" H 7150 4950 50  0001 C CNN
@@
 P 2600 4100
 F 0 "C16" H 2715 4146 50  0000 L CNN
-F 1 "4.7n" H 2715 4055 50  0000 L CNN
+F 1 "10uF" H 2715 4055 50  0000 L CNN
 F 2 "Capacitors_SMD:C_0805" H 2638 3950 50  0001 C CNN
 F 3 "~" H 2600 4100 50  0001 C CNN
@@
 Wire Wire Line
 	2600 3100 3150 3100
-Wire Wire Line
-	3800 3800 4350 3800
 Text Label 4400 3800 0    50   ~ 0
 LED_VCC
-$Comp
-L Device:R R22
-U 1 1 5B369139
-P 4350 4100
-F 0 "R22" H 4420 4146 50  0000 L CNN
-F 1 "100k" H 4420 4055 50  0000 L CNN
-F 2 "Resistors_SMD:R_0805" V 4280 4100 50  0001 C CNN
-F 3 "~" H 4350 4100 50  0001 C CNN
-	1    4350 4100
-	1    0    0    -1
-$EndComp
-Wire Wire Line
-	4350 4250 4350 4350
-Wire Wire Line
-	4350 4350 3950 4350
-Connection ~ 3950 4350
-Wire Wire Line
-	4350 3800 4350 3950
-Connection ~ 4350 3800
-Wire Wire Line
-	4350 3800 4400 3800
 $Comp
 L power:+5V #PWR0154
@@
 Text Label 8500 1500 0    50   ~ 0
 OPAMP_GND
+Wire Wire Line
+	3800 3800 4400 3800
+Text Notes 6200 2150 0    51   ~ 0
+~~1.95V here
 $EndSCHEMATC

Commit message: Imported flag shape into outline layer & finished layout
Parts:
- added TP10: TP_339+_BLUE, my-footprints:Test_Point_1mm, symbol Connector_Specialized:Test_Point
- added TP11: TP_339+_GREEN, my-footprints:Test_Point_1mm, symbol Connector_Specialized:Test_Point
- added TP12: TP_339+_YELLOW, my-footprints:Test_Point_1mm, symbol Connector_Specialized:Test_Point
- added TP13: TP_555THRES, my-footprints:Test_Point_1mm, symbol Connector_Specialized:Test_Point
- added TP14: TP_555OUT, my-footprints:Test_Point_1mm, symbol Connector_Specialized:Test_Point
- added TP15: TP_339+_ORANGE, my-footprints:Test_Point_1mm, symbol Connector_Specialized:Test_Point
- added TP16: TP_339-, my-footprints:Test_Point_1mm, symbol Connector_Specialized:Test_Point
- added TP27: TP_GND, my-footprints:Test_Point_1mm, symbol Connector_Specialized:Test_Point
- added TP30: TP_555TRIG, my-footprints:Test_Point_1mm, symbol Connector_Specialized:Test_Point
- C16: value 10uF -> 10µF
- SW6: footprint my-footprints:Tiny_SMD_Side_Btn_4x2.5mm -> my-footprints:Btn_SMD_6x3.5mm
Connections:
- wire segments 87 -> 93
Changed lines of the file:
@@
 P 2600 4100
 F 0 "C16" H 2715 4146 50  0000 L CNN
-F 1 "10uF" H 2715 4055 50  0000 L CNN
+F 1 "10µF" H 2715 4055 50  0000 L CNN
 F 2 "Capacitors_SMD:C_0805" H 2638 3950 50  0001 C CNN
 F 3 "~" H 2600 4100 50  0001 C CNN
@@
 	2600 3950 2600 3800
 Wire Wire Line
-	2600 3800 2750 3800
+	2600 3800 2650 3800
 Wire Wire Line
 	2600 4250 2600 4350
@@
 F 0 "SW6" V 2150 4450 50  0000 R CNN
 F 1 "SW_SeeBattGauge" V 2250 4850 50  0000 R CNN
-F 2 "my-footprints:Tiny_SMD_Side_Btn_4x2.5mm" H 2100 4300 50  0001 C CNN
+F 2 "my-footprints:Btn_SMD_6x3.5mm" H 2100 4300 50  0001 C CNN
 F 3 "" H 2100 4300 50  0001 C CNN
 	1    2100 4100
@@
 	2100 3750 2100 3900
 Wire Wire Line
-	2100 3900 2750 3900
+	2100 3900 2150 3900
 Connection ~ 2100 3900
 Wire Wire Line
@@
 	6700 4100 6700 4500
 Wire Wire Line
-	6700 2150 6950 2150
+	6700 2150 6850 2150
 Wire Wire Line
 	6950 2150 6950 2300
@@
 	6700 4500 6700 4600
 Wire Wire Line
-	7150 5150 7450 5150
+	7150 5150 7400 5150
 Wire Wire Line
 	7450 5150 7450 4850
@@
 OPAMP_GND
 Wire Wire Line
-	3800 3800 4400 3800
+	3800 3800 3900 3800
 Text Notes 6200 2150 0    51   ~ 0
 ~~1.95V here
+$Comp
+L Connector_Specialized:Test_Point TP14
+U 1 1 5B4F334B
+P 3900 3800
+F 0 "TP14" H 3958 3920 50  0000 L CNN
+F 1 "TP_555OUT" H 3958 3829 50  0000 L CNN
+F 2 "my-footprints:Test_Point_1mm" H 4100 3800 50  0001 C CNN
+F 3 "~" H 4100 3800 50  0001 C CNN
+	1    3900 3800
+	1    0    0    -1
+$EndComp
+Connection ~ 3900 3800
+Wire Wire Line
+	3900 3800 4400 3800
+$Comp
+L Connector_Specialized:Test_Point TP10
+U 1 1 5B4F37C5
+P 6850 2150
+F 0 "TP10" H 6908 2270 50  0000 L CNN
+F 1 "TP_339+_BLUE" H 6908 2179 50  0000 L CNN
+F 2 "my-footprints:Test_Point_1mm" H 7050 2150 50  0001 C CNN
+F 3 "~" H 7050 2150 50  0001 C CNN
+	1    6850 2150
+	1    0    0    -1
+$EndComp
+Connection ~ 6850 2150
+Wire Wire Line
+	6850 2150 6950 2150
+$Comp
+L Connector_Specialized:Test_Point TP11
+U 1 1 5B4F3EB9
+P 6950 3000
+F 0 "TP11" H 7008 3120 50  0000 L CNN
+F 1 "TP_339+_GREEN" H 7008 3029 50  0000 L CNN
+F 2 "my-footprints:Test_Point_1mm" H 7150 3000 50  0001 C CNN
+F 3 "~" H 7150 3000 50  0001 C CNN
+	1    6950 3000
+	1    0    0    -1
+$EndComp
+Connection ~ 6950 3000
+$Comp
+L Connector_Specialized:Test_Point TP12
+U 1 1 5B4F3F53
+P 6950 3750
+F 0 "TP12" H 7008 3870 50  0000 L CNN
+F 1 "TP_339+_YELLOW" H 7008 3779 50  0000 L CNN
+F 2 "my-footprints:Test_Point_1mm" H 7150 3750 50  0001 C CNN
+F 3 "~" H 7150 3750 50  0001 C CNN
+	1    6950 3750
+	1    0    0    -1
+$EndComp
+Connection ~ 6950 3750
+$Comp
+L Connector_Specialized:Test_Point TP15
+U 1 1 5B4F3FCD
+P 6950 4500
+F 0 "TP15" H 7008 4620 50  0000 L CNN
+F 1 "TP_339+_ORANGE" H 7008 4529 50  0000 L CNN
+F 2 "my-footprints:Test_Point_1mm" H 7150 4500 50  0001 C CNN
+F 3 "~" H 7150 4500 50  0001 C CNN
+	1    6950 4500
+	1    0    0    -1
+$EndComp
+Connection ~ 6950 4500
+$Comp
+L Connector_Specialized:Test_Point TP16
+U 1 1 5B4F4047
+P 7400 5150
+F 0 "TP16" H 7458 5270 50  0000 L CNN
+F 1 "TP_339-" H 7458 5179 50  0000 L CNN
+F 2 "my-footprints:Test_Point_1mm" H 7600 5150 50  0001 C CNN
+F 3 "~" H 7600 5150 50  0001 C CNN
+	1    7400 5150
+	1    0    0    -1
+$EndComp
+Connection ~ 7400 5150
+Wire Wire Line
+	7400 5150 7450 5150
+$Comp
+L Connector_Specialized:Test_Point TP13
+U 1 1 5B50A1EA
+P 2650 3800
+F 0 "TP13" H 2708 3920 50  0000 L CNN
+F 1 "TP_555THRES" H 2708 3829 50  0000 L CNN
+F 2 "my-footprints:Test_Point_1mm" H 2850 3800 50  0001 C CNN
+F 3 "~" H 2850 3800 50  0001 C CNN
+	1    2650 3800
+	1    0    0    -1
+$EndComp
+Connection ~ 2650 3800
+Wire Wire Line
+	2650 3800 2750 3800
+$Comp
+L Connector_Specialized:Test_Point TP27
+U 1 1 5B45B9D4
+P 4250 1350
+F 0 "TP27" H 4308 1470 50  0000 L CNN
+F 1 "TP_GND" H 4308 1379 50  0000 L CNN
+F 2 "my-footprints:Test_Point_1mm" H 4450 1350 50  0001 C CNN
+F 3 "~" H 4450 1350 50  0001 C CNN
+	1    4250 1350
+	1    0    0    -1
+$EndComp
+Wire Wire Line
+	4250 1350 4050 1350
+$Comp
+L Connector_Specialized:Test_Point TP30
+U 1 1 5B47E5AE
+P 2150 3900
+F 0 "TP30" H 2208 4020 50  0000 L CNN
+F 1 "TP_555TRIG" H 2208 3929 50  0000 L CNN
+F 2 "my-footprints:Test_Point_1mm" H 2350 3900 50  0001 C CNN
+F 3 "~" H 2350 3900 50  0001 C CNN
+	1    2150 3900
+	1    0    0    -1
+$EndComp
+Connection ~ 2150 3900
+Wire Wire Line
+	2150 3900 2750 3900
 $EndSCHEMATC
