File: MCU_LED-Driver.sch (KiCad schematic (older format))
At the start: 30 parts

Commit message: Schematics complete, ready for prototype PCBs to be designed
Parts:
- removed C?: C, symbol Device:C
- removed D?: LED_Boot_Yellow, symbol Device:LED_Small
- removed D?: LED_Err_Red, symbol Device:LED_Small
- removed R? (x2): R, symbol Device:R
- added C10: 4.7uF, Capacitors_SMD:C_0805, symbol Device:C
- added C11: 10nF, Capacitors_SMD:C_0805, symbol Device:C
- added C12, C14: 1uF, Capacitors_SMD:C_0805, symbol Device:C
- added C13, C15, C9: 100nF, Capacitors_SMD:C_0805, symbol Device:C
- added J4: Conn_SWD20, Pin_Headers:Pin_Header_Straight_2x10_Pitch2.54mm_SMD, symbol Connector_Generic:Conn_02x10_Odd_Even
- added R10, R9: 4k7, Resistors_SMD:R_0805, symbol Device:R
- added R11: 100k, Resistors_SMD:R_0805, symbol Device:R
- added R12: 3k9, Resistors_SMD:R_0805, symbol Device:R
- DA1, DA2, DA3, DB1, DB2, DB3, DC1, DC2, DC3, DD1, DD2, DD3, DE1, DE2, DE3, DF1, DF2, DF3: renamed from D?; footprint (none) -> Diodes_SMD:D_0805
- SW2, SW3, SW4: renamed from SW?; footprint (none) -> my-footprints:Tiny_SMD_Side_Btn_4x2.5mm
- SW5: renamed from SW?; footprint (none) -> Buttons_Switches_SMD:SW_SPDT_PCM12
- U8: renamed from U?; footprint (none) -> SMD_Packages:SOIC-24
- gave numbers to parts that had none: 2
Connections:
- net labels added: RESET, SWCLK, SWDIO
- wire segments 73 -> 129
- no-connect marks 0 -> 4
Other:
- note added: "GND to boot normally;\n3V3 to boot to bootloader"
- note added: "Max LED current is:\nI_max = 58.5 * (1.3 / R_ext)\n\nR_ext = 3k3 => 23mA\nR_ext = 3k6 => 21mA\nR_ext = 3k9 => 19.5mA"

Commit message: Prototype PCB laid out, no tracks yet
Parts:
- J3: footprint Connector_PinHeader_1.27mm:PinHeader_2x05_P1.27mm_Vertical_SMD -> Pin_Headers:Pin_Header_Straight_2x05_Pitch1.27mm_SMD
- U7: footprint Package_SO:TSSOP-20_4.4x6.5mm_P0.65mm -> digikey-footprints:SOIC-24_W7.50mm
Changed lines of the file:
@@
 F 0 "U7" H 9500 3500 50  0000 C CNN
 F 1 "STM32F042F6P6" H 8800 3500 50  0000 C CNN
-F 2 "Package_SO:TSSOP-20_4.4x6.5mm_P0.65mm" H 9600 3425 50  0001 R TNN
+F 2 "digikey-footprints:SOIC-24_W7.50mm" H 9600 3425 50  0001 R TNN
 F 3 "http://www.st.com/st-web-ui/static/active/en/resource/technical/document/datasheet/DM00105814.pdf" H 6800 2550 50  0001 C CNN
 	1    6800 2550
@@
 F 0 "J3" H 1400 3000 50  0000 R CNN
 F 1 "SWD_Conn" H 950 3000 50  0000 R CNN
-F 2 "Connector_PinHeader_1.27mm:PinHeader_2x05_P1.27mm_Vertical_SMD" H 1100 1900 50  0001 L TNN
+F 2 "Pin_Headers:Pin_Header_Straight_2x05_Pitch1.27mm_SMD" H 1100 1900 50  0001 L TNN
 F 3 "http://infocenter.arm.com/help/topic/com.arm.doc.faqs/attached/13634/cortex_debug_connectors.pdf" V 700 1200 50  0001 C CNN
 	1    1050 2450

Commit message: Prototype PCB design finished?
Connections:
- net labels added: USBDM, USBDP
- net labels removed: USB_D+, USB_D-
- wire segments 129 -> 131
Changed lines of the file:
@@
 $Descr A4 11693 8268
 encoding utf-8
-Sheet 3 4
+Sheet 4 4
 Title ""
 Date ""
@@
 Text HLabel 5400 600  2    50   Input ~ 0
 GND
-Text HLabel 9700 2850 2    50   Input ~ 0
-USB_D+
-Text HLabel 9700 2750 2    50   Input ~ 0
-USB_D-
 $Comp
 L power:+5V #PWR0124
@@
 Wire Wire Line
 	10850 2050 10850 2100
+Wire Wire Line
+	10000 2750 9700 2750
+Wire Wire Line
+	9700 2850 10000 2850
+Text GLabel 10000 2750 2    50   BiDi ~ 0
+USBDP
+Text GLabel 10000 2850 2    50   BiDi ~ 0
+USBDM
 $EndSCHEMATC

Commit message: Fixed footprints for a few ICs. Oops.
Updated PCB layout to come!
Parts:
- U7: footprint digikey-footprints:SOIC-24_W7.50mm -> digikey-footprints:TSSOP-20_W4.4mm
- U8: footprint SMD_Packages:SOIC-24 -> digikey-footprints:SOIC-24_W7.50mm
Changed lines of the file:
@@
 F 0 "U8" H 3425 6187 60  0000 C CNN
 F 1 "IS31FL3218" H 3425 6081 60  0000 C CNN
-F 2 "SMD_Packages:SOIC-24" H 3400 5350 60  0001 C CNN
+F 2 "digikey-footprints:SOIC-24_W7.50mm" H 3400 5350 60  0001 C CNN
 F 3 "G:/Andrew/Google Drive/Electronics/_Documentation/Hardware data sheets/ISSI 31FL 3218 18ch PWM LED driver.pdf" H 3400 5350 60  0001 C CNN
 	1    3400 5350
@@
 F 0 "U7" H 9500 3500 50  0000 C CNN
 F 1 "STM32F042F6P6" H 8800 3500 50  0000 C CNN
-F 2 "digikey-footprints:SOIC-24_W7.50mm" H 9600 3425 50  0001 R TNN
+F 2 "digikey-footprints:TSSOP-20_W4.4mm" H 9600 3425 50  0001 R TNN
 F 3 "http://www.st.com/st-web-ui/static/active/en/resource/technical/document/datasheet/DM00105814.pdf" H 6800 2550 50  0001 C CNN
 	1    6800 2550

Commit message: More fixes after testing the LED gauge and such
Parts:
- removed R11: 100k, Resistors_SMD:R_0805, symbol Device:R
Connections:
- wire segments 131 -> 129
Changed lines of the file:
@@
-$EndComp
-$Comp
-L Device:R R11
-U 1 1 5B3980DF
-P 2450 6550
-F 0 "R11" H 2520 6596 50  0000 L CNN
-F 1 "100k" H 2520 6505 50  0000 L CNN
-F 2 "Resistors_SMD:R_0805" V 2380 6550 50  0001 C CNN
-F 3 "~" H 2450 6550 50  0001 C CNN
-	1    2450 6550
-	1    0    0    -1
 $EndComp
 $Comp
@@
 Wire Wire Line
 	2650 7550 2900 7550
-Wire Wire Line
-	2450 6400 2450 6350
-Wire Wire Line
-	2450 6350 2900 6350
 Wire Wire Line
 	1850 5950 1850 6050
@@
 Wire Wire Line
 	2500 5300 2700 5300
-$Comp
-L power:GND #PWR0136
-U 1 1 5B3B0C32
-P 2450 6700
-F 0 "#PWR0136" H 2450 6450 50  0001 C CNN
-F 1 "GND" H 2455 6527 50  0000 C CNN
-F 2 "" H 2450 6700 50  0001 C CNN
-F 3 "" H 2450 6700 50  0001 C CNN
-	1    2450 6700
-	1    0    0    -1
-$EndComp
 Text Notes 2500 7500 2    51   ~ 0
 Max LED current is:\nI_max = 58.5 * (1.3 / R_ext)\n\nR_ext = 3k3 => 23mA\nR_ext = 3k6 => 21mA\nR_ext = 3k9 => 19.5mA

Commit message: More fixes after prototyping & reading more datasheets
Parts:
- added R11: 100k, Resistors_SMD:R_0805, symbol Device:R
Connections:
- net labels added: ISSI_SDB
- wire segments 129 -> 133
Changed lines of the file:
@@
 Wire Wire Line
 	9700 2850 10000 2850
+Text GLabel 10000 2850 2    50   BiDi ~ 0
+USBDP
 Text GLabel 10000 2750 2    50   BiDi ~ 0
-USBDP
-Text GLabel 10000 2850 2    50   BiDi ~ 0
 USBDM
+$Comp
+L Device:R R11
+U 1 1 5B3E8A83
+P 2550 6550
+F 0 "R11" H 2620 6596 50  0000 L CNN
+F 1 "100k" H 2620 6505 50  0000 L CNN
+F 2 "Resistors_SMD:R_0805" V 2480 6550 50  0001 C CNN
+F 3 "~" H 2550 6550 50  0001 C CNN
+	1    2550 6550
+	1    0    0    -1
+$EndComp
+Connection ~ 2550 6350
+Wire Wire Line
+	2550 6350 2900 6350
+Wire Wire Line
+	1700 6350 2550 6350
+Text Label 1700 6350 2    50   ~ 0
+ISSI_SDB
+Text Label 9700 2250 0    50   ~ 0
+ISSI_SDB
+$Comp
+L power:GND #PWR0136
+U 1 1 5B3F9646
+P 2550 6750
+F 0 "#PWR0136" H 2550 6500 50  0001 C CNN
+F 1 "GND" H 2555 6577 50  0000 C CNN
+F 2 "" H 2550 6750 50  0001 C CNN
+F 3 "" H 2550 6750 50  0001 C CNN
+	1    2550 6750
+	1    0    0    -1
+$EndComp
+Wire Wire Line
+	2550 6750 2550 6700
+Wire Wire Line
+	2550 6400 2550 6350
 $EndSCHEMATC

Commit message: Hopefully final schematic fixes
Parts:
- removed J3: SWD_Conn, Pin_Headers:Pin_Header_Straight_2x05_Pitch1.27mm_SMD, symbol Connector_Specialized:Conn_ARM_JTAG_SWD_10
- removed J4: Conn_SWD20, Pin_Headers:Pin_Header_Straight_2x10_Pitch2.54mm_SMD, symbol Connector_Generic:Conn_02x10_Odd_Even
- added J3: Custom_SWD, Socket_Strips:Socket_Strip_Straight_1x05_Pitch2.00mm, symbol Connector_Generic:Conn_01x05
Connections:
- wire segments 133 -> 114
- no-connect marks 4 -> 0
Changed lines of the file:
@@
 L Switch:SW_Push SW4
 U 1 1 5B3B0E4A
-P 2250 2550
-F 0 "SW4" H 2250 2835 50  0000 C CNN
-F 1 "Reset_BTN" H 2250 2744 50  0000 C CNN
-F 2 "my-footprints:Tiny_SMD_Side_Btn_4x2.5mm" H 2250 2750 50  0001 C CNN
-F 3 "" H 2250 2750 50  0001 C CNN
-	1    2250 2550
+P 3150 2150
+F 0 "SW4" H 3150 2435 50  0000 C CNN
+F 1 "Reset_BTN" H 3150 2344 50  0000 C CNN
+F 2 "my-footprints:Tiny_SMD_Side_Btn_4x2.5mm" H 3150 2350 50  0001 C CNN
+F 3 "" H 3150 2350 50  0001 C CNN
+	1    3150 2150
 	0    -1   -1   0
 $EndComp
@@
 $EndComp
 $Comp
-L Connector_Specialized:Conn_ARM_JTAG_SWD_10 J3
-U 1 1 5B37C53A
-P 1050 2450
-F 0 "J3" H 1400 3000 50  0000 R CNN
-F 1 "SWD_Conn" H 950 3000 50  0000 R CNN
-F 2 "Pin_Headers:Pin_Header_Straight_2x05_Pitch1.27mm_SMD" H 1100 1900 50  0001 L TNN
-F 3 "http://infocenter.arm.com/help/topic/com.arm.doc.faqs/attached/13634/cortex_debug_connectors.pdf" V 700 1200 50  0001 C CNN
-	1    1050 2450
-	1    0    0    -1
-$EndComp
-$Comp
-L power:+3.3V #PWR0131
-U 1 1 5B37F058
-P 1050 1800
-F 0 "#PWR0131" H 1050 1650 50  0001 C CNN
-F 1 "+3.3V" H 1065 1973 50  0000 C CNN
-F 2 "" H 1050 1800 50  0001 C CNN
-F 3 "" H 1050 1800 50  0001 C CNN
-	1    1050 1800
-	1    0    0    -1
-$EndComp
-$Comp
-L power:GND #PWR0132
-U 1 1 5B37F09F
-P 1000 3100
-F 0 "#PWR0132" H 1000 2850 50  0001 C CNN
-F 1 "GND" H 1005 2927 50  0000 C CNN
-F 2 "" H 1000 3100 50  0001 C CNN
-F 3 "" H 1000 3100 50  0001 C CNN
-	1    1000 3100
-	1    0    0    -1
-$EndComp
-Wire Wire Line
-	1550 2150 2250 2150
-Wire Wire Line
-	2550 2150 2550 1950
-Wire Wire Line
-	2550 1950 3900 1950
-Wire Wire Line
-	1050 1800 1050 1850
-Wire Wire Line
-	950  3050 1000 3050
-Wire Wire Line
-	1000 3050 1000 3100
-Connection ~ 1000 3050
-Wire Wire Line
-	1000 3050 1050 3050
-$Comp
 L Device:C C10
 U 1 1 5B392F81
@@
 L Device:C C13
 U 1 1 5B3BA212
-P 2550 2550
-F 0 "C13" H 2665 2596 50  0000 L CNN
-F 1 "100nF" H 2665 2505 50  0000 L CNN
-F 2 "Capacitors_SMD:C_0805" H 2588 2400 50  0001 C CNN
-F 3 "~" H 2550 2550 50  0001 C CNN
-	1    2550 2550
-	1    0    0    -1
-$EndComp
-Wire Wire Line
-	2550 2400 2550 2350
-Wire Wire Line
-	2550 2350 2250 2350
-Wire Wire Line
-	2550 2700 2550 2750
-Wire Wire Line
-	2550 2750 2250 2750
-Wire Wire Line
-	2250 2350 2250 2150
-Connection ~ 2250 2350
-Connection ~ 2250 2150
-Wire Wire Line
-	2250 2150 2550 2150
+P 3450 2150
+F 0 "C13" H 3565 2196 50  0000 L CNN
+F 1 "100nF" H 3565 2105 50  0000 L CNN
+F 2 "Capacitors_SMD:C_0805" H 3488 2000 50  0001 C CNN
+F 3 "~" H 3450 2150 50  0001 C CNN
+	1    3450 2150
+	1    0    0    -1
+$EndComp
+Wire Wire Line
+	3450 2000 3450 1950
+Wire Wire Line
+	3450 1950 3150 1950
+Wire Wire Line
+	3450 2300 3450 2350
+Wire Wire Line
+	3450 2350 3150 2350
 $Comp
 L power:GND #PWR0137
 U 1 1 5B3C2765
-P 2250 2750
-F 0 "#PWR0137" H 2250 2500 50  0001 C CNN
-F 1 "GND" H 2255 2577 50  0000 C CNN
-F 2 "" H 2250 2750 50  0001 C CNN
-F 3 "" H 2250 2750 50  0001 C CNN
-	1    2250 2750
-	1    0    0    -1
-$EndComp
-Connection ~ 2250 2750
+P 3150 2350
+F 0 "#PWR0137" H 3150 2100 50  0001 C CNN
+F 1 "GND" H 3155 2177 50  0000 C CNN
+F 2 "" H 3150 2350 50  0001 C CNN
+F 3 "" H 3150 2350 50  0001 C CNN
+	1    3150 2350
+	1    0    0    -1
+$EndComp
+Connection ~ 3150 2350
 $Comp
 L power:GND #PWR0138
@@
 Text Notes 4200 3750 0    51   ~ 0
 GND to boot normally;\n3V3 to boot to bootloader
-$Comp
-L Connector_Generic:Conn_02x10_Odd_Even J4
-U 1 1 5B415BA3
-P 10400 5700
-F 0 "J4" H 10450 6317 50  0000 C CNN
-F 1 "Conn_SWD20" H 10450 6226 50  0000 C CNN
-F 2 "Pin_Headers:Pin_Header_Straight_2x10_Pitch2.54mm_SMD" H 10400 5700 50  0001 C CNN
-F 3 "~" H 10400 5700 50  0001 C CNN
-	1    10400 5700
-	1    0    0    -1
-$EndComp
 Text Label 3800 1950 2    51   ~ 0
 RESET
@@
 Text Label 9700 3050 0    51   ~ 0
 SWCLK
-$Comp
-L power:+3.3V #PWR0143
-U 1 1 5B41742C
-P 10000 5300
-F 0 "#PWR0143" H 10000 5150 50  0001 C CNN
-F 1 "+3.3V" H 10015 5473 50  0000 C CNN
-F 2 "" H 10000 5300 50  0001 C CNN
-F 3 "" H 10000 5300 50  0001 C CNN
-	1    10000 5300
-	1    0    0    -1
-$EndComp
-$Comp
-L power:GND #PWR0144
-U 1 1 5B417493
-P 9850 5350
-F 0 "#PWR0144" H 9850 5100 50  0001 C CNN
-F 1 "GND" H 9855 5177 50  0000 C CNN
-F 2 "" H 9850 5350 50  0001 C CNN
-F 3 "" H 9850 5350 50  0001 C CNN
-	1    9850 5350
-	1    0    0    -1
-$EndComp
-$Comp
-L power:GND #PWR0145
-U 1 1 5B417AB6
-P 10800 6250
-F 0 "#PWR0145" H 10800 6000 50  0001 C CNN
-F 1 "GND" H 10805 6077 50  0000 C CNN
-F 2 "" H 10800 6250 50  0001 C CNN
-F 3 "" H 10800 6250 50  0001 C CNN
-	1    10800 6250
-	1    0    0    -1
-$EndComp
-Wire Wire Line
-	10800 6250 10800 6200
-Wire Wire Line
-	10800 6200 10700 6200
-Wire Wire Line
-	10700 6200 10700 6100
-Connection ~ 10700 6200
-Connection ~ 10700 5500
-Wire Wire Line
-	10700 5500 10700 5400
-Connection ~ 10700 5600
-Wire Wire Line
-	10700 5600 10700 5500
-Connection ~ 10700 5700
-Wire Wire Line
-	10700 5700 10700 5600
-Connection ~ 10700 5800
-Wire Wire Line
-	10700 5800 10700 5700
-Connection ~ 10700 5900
-Wire Wire Line
-	10700 5900 10700 5800
-Connection ~ 10700 6000
-Wire Wire Line
-	10700 6000 10700 5900
-Connection ~ 10700 6100
-Wire Wire Line
-	10700 6100 10700 6000
-$Comp
-L power:+3.3V #PWR0146
-U 1 1 5B421AFD
-P 10850 5300
-F 0 "#PWR0146" H 10850 5150 50  0001 C CNN
-F 1 "+3.3V" H 10865 5473 50  0000 C CNN
-F 2 "" H 10850 5300 50  0001 C CNN
-F 3 "" H 10850 5300 50  0001 C CNN
-	1    10850 5300
-	1    0    0    -1
-$EndComp
-Wire Wire Line
-	10850 5300 10700 5300
-Wire Wire Line
-	9850 5350 9950 5350
-Wire Wire Line
-	9950 5350 9950 5400
-Wire Wire Line
-	9950 5400 10200 5400
-Wire Wire Line
-	10200 5400 10200 5500
-Connection ~ 10200 5400
-Text Label 10200 6000 2    51   ~ 0
-RESET
-Text Label 10200 5600 2    51   ~ 0
-SWDIO
-Text Label 10200 5700 2    51   ~ 0
-SWCLK
-NoConn ~ 10200 5800
-NoConn ~ 10200 5900
-NoConn ~ 10200 6100
-NoConn ~ 10200 6200
-Wire Wire Line
-	10000 5300 10200 5300
 $Comp
 L power:GND #PWR0147
@@
 Wire Wire Line
 	2550 6400 2550 6350
+$Comp
+L Connector_Generic:Conn_01x05 J3
+U 1 1 5B487F17
+P 10400 5900
+F 0 "J3" H 10480 5942 50  0000 L CNN
+F 1 "Custom_SWD" H 10480 5851 50  0000 L CNN
+F 2 "Socket_Strips:Socket_Strip_Straight_1x05_Pitch2.00mm" H 10400 5900 50  0001 C CNN
+F 3 "~" H 10400 5900 50  0001 C CNN
+	1    10400 5900
+	1    0    0    -1
+$EndComp
+$Comp
+L power:+3.3V #PWR0132
+U 1 1 5B487FC9
+P 10100 5700
+F 0 "#PWR0132" H 10100 5550 50  0001 C CNN
+F 1 "+3.3V" H 10115 5873 50  0000 C CNN
+F 2 "" H 10100 5700 50  0001 C CNN
+F 3 "" H 10100 5700 50  0001 C CNN
+	1    10100 5700
+	1    0    0    -1
+$EndComp
+$Comp
+L power:GND #PWR0143
+U 1 1 5B488020
+P 10100 6100
+F 0 "#PWR0143" H 10100 5850 50  0001 C CNN
+F 1 "GND" H 10105 5927 50  0000 C CNN
+F 2 "" H 10100 6100 50  0001 C CNN
+F 3 "" H 10100 6100 50  0001 C CNN
+	1    10100 6100
+	1    0    0    -1
+$EndComp
+Text Label 10100 5800 2    51   ~ 0
+SWDIO
+Text Label 10100 5900 2    51   ~ 0
+SWCLK
+Text Label 10100 6000 2    51   ~ 0
+RESET
+Wire Wire Line
+	10100 5700 10200 5700
+Wire Wire Line
+	10200 5800 10100 5800
+Wire Wire Line
+	10100 5900 10200 5900
+Wire Wire Line
+	10200 6000 10100 6000
+Wire Wire Line
+	10100 6100 10200 6100
+Connection ~ 3450 1950
+Wire Wire Line
+	3450 1950 3900 1950
 $EndSCHEMATC

Commit message: Imported flag shape into outline layer & finished layout
Parts:
- removed SW5: Boot_SW, Buttons_Switches_SMD:SW_SPDT_PCM12, symbol Switch:SW_DPDT_x2
- added D9: LED_Small, LEDs:LED_0805, symbol Device:LED_Small
- added R28: 2k7, Resistors_SMD:R_0805, symbol Device:R
- added R29: 10k, Resistors_SMD:R_0805, symbol Device:R
- added SW5: Boot_BTN, my-footprints:Tiny_SMD_Side_Btn_4x2.5mm, symbol Switch:SW_Push
- added TP17: TP_MODEBTN, my-footprints:Test_Point_1mm, symbol Connector_Specialized:Test_Point
- added TP18: TP_BRIGHTBTN, my-footprints:Test_Point_1mm, symbol Connector_Specialized:Test_Point
- added TP19: TP_SWDIO, my-footprints:Test_Point_1mm, symbol Connector_Specialized:Test_Point
- added TP20: TP_SWCLK, my-footprints:Test_Point_1mm, symbol Connector_Specialized:Test_Point
- added TP21, TP25: TP_~RST, my-footprints:Test_Point_1mm, symbol Connector_Specialized:Test_Point
- added TP22: TP_SDA, my-footprints:Test_Point_1mm, symbol Connector_Specialized:Test_Point
- added TP23: TP_SCL, my-footprints:Test_Point_1mm, symbol Connector_Specialized:Test_Point
- added TP24: TP_IS_SDB, my-footprints:Test_Point_1mm, symbol Connector_Specialized:Test_Point
- added TP26: TP_BOOT, my-footprints:Test_Point_1mm, symbol Connector_Specialized:Test_Point
- added TP28: TP_GND, my-footprints:Test_Point_1mm, symbol Connector_Specialized:Test_Point
- added TP29: TP_3V3, my-footprints:Test_Point_1mm, symbol Connector_Specialized:Test_Point
- C10: value 4.7uF -> 4.7µF
- C12, C14: value 1uF -> 1µF
- J3: footprint Socket_Strips:Socket_Strip_Straight_1x05_Pitch2.00mm -> w_smd_strip:bb02-hy05a
- SW2, SW3: footprint my-footprints:Tiny_SMD_Side_Btn_4x2.5mm -> my-footprints:Btn_SMD_6x3.5mm
Connections:
- wire segments 114 -> 135
